File: MCP251863Breakout.kicad_pcb (KiCad board)
At the start: 2 copper layers, 32 x 32 mm, 27 parts, among them U1 MCP251863T-H-SS, U2 AMS1117-3.3, Y1 Crystal_GND24

Commit message: Break out STBY to a pad, add GND/PWR pads beside CANL/CANH, set LCSC basic parts
- U1 STBY (pin 5) no longer tied to GND: new STBY pad below CS, routed on B.Cu
- GND2 left of CANL, PWR2 (+5V, to C12) right of CANH
- LCSC: C96446 10u, C14663 100n, C1634 10p, C22787 120R, C6186 AMS1117
- Schematic test-pad refs match the board (clears parity), rev 1.1
- Regenerated production files, PDF, renders, README
Parts:
- added GND2: TestPoint_Square, TestPoint:TestPoint_Pad_2.0x2.0mm, F.Cu at (143.8, 92.0)
- added PWR2: TestPoint_Square, TestPoint:TestPoint_Pad_2.0x2.0mm, F.Cu at (161.5, 92.0)
- added STBY: TestPoint_Square, TestPoint:TestPoint_Pad_2.0x2.0mm, F.Cu at (136.5, 118.5)
Connections:
- U1 pad 5: GND -> /STBY
Routing:
- net /STBY: track 0.00 -> 32.2 mm, vias 0 -> 2
- net GND: track 15.9 -> 9.98 mm, vias 58 -> 46
- net +5V: track 34.9 -> 39.4 mm
