File: MCP251863Breakout.kicad_sch (KiCad schematic)
At the start: 27 parts, among them U1 MCP251863T-H-SS, U2 AMS1117-3.3, Y1 Crystal_GND24

Commit message: Break out STBY to a pad, add GND/PWR pads beside CANL/CANH, set LCSC basic parts
- U1 STBY (pin 5) no longer tied to GND: new STBY pad below CS, routed on B.Cu
- GND2 left of CANL, PWR2 (+5V, to C12) right of CANH
- LCSC: C96446 10u, C14663 100n, C1634 10p, C22787 120R, C6186 AMS1117
- Schematic test-pad refs match the board (clears parity), rev 1.1
- Regenerated production files, PDF, renders, README
Parts:
- added GND2, PWR2, STBY: TestPoint_Square, TestPoint:TestPoint_Pad_2.0x2.0mm, symbol Connector:TestPoint_Square
- C1, C10, C12, C4: LCSC Part (none) -> C96446
- C2, C3, C5, C6, C7: LCSC Part (none) -> C14663
- C8, C9: LCSC Part (none) -> C1634
- R1: LCSC Part (none) -> C22787
- U2: LCSC Part (none) -> C6186
- renumbered CANH1 to CANH, CANL1 to CANL, CLKO1 to CLKO, CS1 to CS, GND1 to GND, INT2 to INT, MISO1 to MISO, MOSI1 to MOSI, PWR1 to PWR, SCK1 to SCK
Connections:
- net +5V: now also PWR2.1
- net GND: now also GND2.1; no longer U1.5 (STBY)
- new net STBY: STBY.1, U1.5 (STBY)
